File: PCB/main.sch (EAGLE design)
At the start: 58 parts, among them X1 BU-SMA-V

Commit message: Eagle Schematic Changes
- Altered headers
- Replaced solder pads with  pin headers
- Connected rec pins
- Added RTC
- Swapped V+ for 5V connections
- Swapped amplifier to 5v supply
Parts:
- removed AUX1: (no value), pinhead:PINHD-1X3
- removed G1, G2, G3, G4, G5, G6, G7, G8, G9: LSP10, solpad:LSP10
- removed REC1: (no value), pinhead:PINHD-2X5
- removed V+: LSP11, solpad:LSP11
- added H13: (no value), pinhead:PINHD-1X2
- added H14, H15, H17: (no value), pinhead:PINHD-1X3
- added H16: (no value), pinhead:PINHD-2X5
- added JP1: (no value), pinhead:PINHD-1X4/90
- H12: device pinhead:PINHD-1X10 -> pinhead:PINHD-1X3
- H8, H9: device pinhead:PINHD-1X3 -> pinhead:PINHD-1X2
- R11, R12: value 330 -> (none)
Connections:
- removed net 10: H12.10
- removed net 2: H12.2
- removed net 3: H12.3
- removed net 7: H12.7
- removed net 9: H12.9
- removed net PIC23: H3.7, MICROCONTROLLER.RA1/AN1
- removed net PIC24: H3.8, MICROCONTROLLER.RA0/AN0
- removed net PIC27: H3.11, MICROCONTROLLER.RA5/AN4/HLVDIN/SEG15
- removed net PIC28: H3.12, MICROCONTROLLER.RA4/T0CKI/SEG14
- removed net PIC36: H2.4, MICROCONTROLLER.RC5/SDO/SEG12
- removed net SDA: H2.3, H6.2, MICROCONTROLLER.RC4/SDI/SDA, R1.2, U$1.SDA, U$2.DATA, U$3.SDA
- new net +5V: AMP-R.V+, C4.1, H15.1, H15.2, H15.3, VOLTAGE_REGULATOR.VIN
- new net BT-L: H17.3, U$3.NO4
- new net BT-R: H17.2, U$1.NO4
- new net DREQ: H16.7, H3.8, MICROCONTROLLER.RA0/AN0
- new net MOSI: H16.5, H2.4, MICROCONTROLLER.RC5/SDO/SEG12
- new net SDA/MISO: H16.4, H2.3, JP1.3, MICROCONTROLLER.RC4/SDI/SDA, R1.2, U$1.SDA, U$2.DATA, U$3.SDA
- new net XCS: H16.9, H3.7, MICROCONTROLLER.RA1/AN1
- new net XDCS: H16.10, H3.12, MICROCONTROLLER.RA4/T0CKI/SEG14
- new net XRST: H16.8, H3.11, MICROCONTROLLER.RA5/AN4/HLVDIN/SEG15
- net +3V3: now also H14.1, H14.2, H14.3, JP1.2; no longer H7.2
- net AMP-L: now also H8.2; no longer H10.3
- net AMP-R: now also H8.1; no longer H10.2
- net AUX-L: now also H10.3, H6.1; no longer AUX1.3, H9.3
- net AUX-R: now also H10.2, H7.1; no longer AUX1.2, H9.2
- net FM-L: now also H13.2, H6.3; no longer H8.3
- net FM-R: now also H13.1, H7.3; no longer H8.2
- net GND: now also H11.2, H11.3, H12.1, H16.3, H17.1, JP1.1; no longer AUX1.1, G1.MP, G2.MP, G3.MP, H6.1, H7.1, H8.1, H9.1
- net L-OUT: now also H9.2; no longer H11.3
- net R-OUT: now also H9.1; no longer H11.2
- net REC-L: now also H12.3, H6.2
- net REC-R: now also H12.2, H7.2
- net SCL: now also H16.6, JP1.4; no longer H6.3
- net V+: now also H16.1, H16.2; no longer AMP-R.V+, C4.1, G7.MP, G8.MP, G9.MP, H12.1, H12.6, H7.3, REC1.1, V+.MP, VOLTAGE_REGULATOR.VIN
Other:
- note added: "* These two might need splitting at PCB design"
- note added: "AMP"
- note added: "AUX"
- note added: "Input headers"
- note added: "Left"
- note added: "Output"
- note added: "REC in"
- note added: "REC out"
- note added: "Real Time Clock"
- note added: "Recorder"
- note added: "Right"
- note added: "Testing headers"
- note removed: "AMP test"
- note removed: "AUX test"
- note removed: "I2C Debug"
- note removed: "Output test"
- note removed: "Radio test"
- note removed: "Recorder test"
- note removed: "Voltage test"
- moved on the sheet: H10, H11, H5, H6, H7, R1, R13, R2
